File: mcu.kicad_sch (KiCad schematic)
At the start: 13 parts, among them J1 Micro_SD_Card, J2 Conn_01x40, J3 USB_C_Receptacle_USB2.0_14P, U1 ESP32-S3-WROOM-1

Commit message: upd
Other:
- moved on the sheet: J2, U1
Changed lines of the file:
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@@
 	(symbol
 		(lib_id "RF_Module:ESP32-S3-WROOM-1")
-		(at 137.16 59.69 0)
+		(at 44.45 60.96 0)
 		(unit 1)
 		(exclude_from_sim no)
@@
 		(fields_autoplaced yes)
 		(property "Reference" "U1"
-			(at 139.3541 29.21 0)
+			(at 46.6441 30.48 0)
 			(effects
 				(font
@@
 		)
 		(property "Value" "ESP32-S3-WROOM-1"
-			(at 139.3541 31.75 0)
+			(at 46.6441 33.02 0)
 			(effects
 				(font
@@
 		)
 		(property "Footprint" "RF_Module:ESP32-S3-WROOM-1"
-			(at 137.16 57.15 0)
+			(at 44.45 58.42 0)
 			(effects
 				(font
@@
 		)
 		(property "Datasheet" "https://www.espressif.com/sites/default/files/documentation/esp32-s3-wroom-1_wroom-1u_datasheet_en.pdf"
-			(at 137.16 59.69 0)
+			(at 44.45 60.96 0)
 			(effects
 				(font
@@
 		)
 		(property "Description" "RF Module, ESP32-S3 SoC, Wi-Fi 802.11b/g/n, Bluetooth, BLE, 32-bit, 3.3V, onboard antenna, SMD"
-			(at 137.16 59.69 0)
+			(at 44.45 60.96 0)
 			(effects
 				(font
@@
 	(symbol
 		(lib_id "Connector_Generic:Conn_01x40")
-		(at 54.61 73.66 0)
+		(at 91.44 71.12 0)
 		(unit 1)
 		(exclude_from_sim no)
@@
 		(fields_autoplaced yes)
 		(property "Reference" "J2"
-			(at 57.15 73.6599 0)
+			(at 93.98 71.1199 0)
 			(effects
 				(font
@@
 		)
 		(property "Value" "Conn_01x40"
-			(at 57.15 76.1999 0)
+			(at 93.98 73.6599 0)
 			(effects
 				(font
@@
 		)
 		(property "Footprint" "Connector_FFC-FPC:Hirose_FH12-40S-0.5SH_1x40-1MP_P0.50mm_Horizontal"
-			(at 54.61 73.66 0)
+			(at 91.44 71.12 0)
 			(effects
 				(font
@@
 		)
 		(property "Datasheet" "~"
-			(at 54.61 73.66 0)
+			(at 91.44 71.12 0)
 			(effects
 				(font
@@
 		)
 		(property "Description" "Generic connector, single row, 01x40, script generated (kicad-library-utils/schlib/autogen/connector/)"
-			(at 54.61 73.66 0)
-			(effects
-				(font
+			(at 91.44 71.12 0)
+			(effects
+				(font
