File: hardware/power.kicad_sch (KiCad schematic)
At the start: 29 parts, among them J5 batt, Q3 Q_NPN_BEC, SW41 SW_SPDT, U4 BQ24075RGT, U5 TLV62569DBV

Commit message: remove ch340
Parts:
- removed Q3: Q_NPN_BEC, symbol Device:Q_NPN_BEC
- added Q4: NPN SS8050, Package_TO_SOT_SMD:SOT-23, symbol Device:Q_NPN_BEC
- R10, R11, R12, R18, R19, R31: footprint (none) -> Resistor_SMD:R_0603_1608Metric
Connections:
- net CHG: now also Q4.3 (C)
- net GND: now also Q4.2 (E)
- net ~{CHG}: now also Q4.1 (B)
Changed lines of the file:
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@@
+	)
+	(symbol
+		(lib_id "Device:Q_NPN_BEC")
+		(at 207.01 139.7 0)
+		(unit 1)
+		(exclude_from_sim no)
+		(in_bom yes)
+		(on_board yes)
+		(dnp no)
+		(fields_autoplaced yes)
+		(property "Reference" "Q4"
+			(at 212.09 138.4299 0)
+			(effects
+				(font
+					(size 1.27 1.27)
+				)
+				(justify left)
+			)
+		)
+		(property "Value" "NPN SS8050"
+			(at 212.09 140.9699 0)
+			(effects
+				(font
+					(size 1.27 1.27)
+				)
+				(justify left)
+			)
+		)
+		(property "Footprint" "Package_TO_SOT_SMD:SOT-23"
+			(at 212.09 137.16 0)
+			(effects
+				(font
+					(size 1.27 1.27)
+				)
+				(hide yes)
+			)
+		)
+		(property "Datasheet" "~"
+			(at 207.01 139.7 0)
+			(effects
+				(font
+					(size 1.27 1.27)
+				)
+				(hide yes)
+			)
+		)
+		(property "Description" "NPN transistor, base/emitter/collector"
+			(at 207.01 139.7 0)
+			(effects
+				(font
+					(size 1.27 1.27)
+				)
+				(hide yes)
+			)
+		)
+		(property "LCSC" "C2150"
+			(at 207.01 139.7 0)
+			(effects
+				(font
+					(size 1.27 1.27)
+				)
+				(hide yes)
+			)
+		)
+		(pin "1"
+		)
+		(pin "3"
+		)
+		(pin "2"
+		)
+		(instances
+			(project "badge"
+				(path "/dc4a3d77-b0f8-4e90-a4be-3e93c7025348/fa1edb42-107e-4301-94d6-2222638475c5"
+					(reference "Q4")
+					(unit 1)
+				)
+			)
+		)
 	)
 	(symbol
@@
 	)
 	(symbol
-		(lib_id "Device:Q_NPN_BEC")
-		(at 207.01 139.7 0)
-		(unit 1)
-		(exclude_from_sim no)
-		(in_bom yes)
-		(on_board yes)
-		(dnp no)
-		(fields_autoplaced yes)
-		(property "Reference" "Q3"
-			(at 212.09 138.4299 0)
-			(effects
-				(font
-					(size 1.27 1.27)
-				)
-				(justify left)
-			)
-		)
-		(property "Value" "Q_NPN_BEC"
-			(at 212.09 140.9699 0)
-			(effects
-				(font
-					(size 1.27 1.27)
-				)
-				(justify left)
-			)
-		)
-		(property "Footprint" ""
-			(at 212.09 137.16 0)
-			(effects
-				(font
-					(size 1.27 1.27)
-				)
-				(hide yes)
-			)
-		)
-		(property "Datasheet" "~"
-			(at 207.01 139.7 0)
-			(effects
-				(font
-					(size 1.27 1.27)
-				)
-				(hide yes)
-			)
-		)
-		(property "Description" "NPN transistor, base/emitter/collector"
-			(at 207.01 139.7 0)
-			(effects
-				(font
-					(size 1.27 1.27)
-				)
-				(hide yes)
-			)
-		)
-		(pin "1"
-		)
-		(pin "3"
-		)
-		(pin "2"
-		)
-		(instances
-			(project "badge"
-				(path "/dc4a3d77-b0f8-4e90-a4be-3e93c7025348/fa1edb42-107e-4301-94d6-2222638475c5"
-					(reference "Q3")
-					(unit 1)
-				)
-			)
-		)
-	)
-	(symbol
 		(lib_id "power:GND")
 		(at 60.96 158.75 0)
@@
 			)
 		)
-		(property "Footprint" ""
+		(property "Footprint" "Resistor_SMD:R_0603_1608Metric"
 			(at 108.458 49.53 90)
 			(effects
@@
 			)
 		)
-		(property "Footprint" ""
+		(property "Footprint" "Resistor_SMD:R_0603_1608Metric"
 			(at 80.772 153.67 90)
 			(effects
@@
 			)
 		)
-		(property "Footprint" ""
+		(property "Footprint" "Resistor_SMD:R_0603_1608Metric"
 			(at 201.168 128.27 90)
 			(effects
@@
 			)
 		)
-		(property "Footprint" ""
+		(property "Footprint" "Resistor_SMD:R_0603_1608Metric"
 			(at 70.612 153.67 90)
 			(effects
@@
 			)
 		)
-		(property "Footprint" ""
+		(property "Footprint" "Resistor_SMD:R_0603_1608Metric"
 			(at 132.842 146.05 90)
 			(effects
@@
 			)
 		)
-		(property "Footprint" ""
+		(property "Footprint" "Resistor_SMD:R_0603_1608Metric"
 			(at 211.328 128.27 90)
 			(effects

Commit message: update usb port, esd, lcsc
Parts:
- renumbered C5 to C2, C2 to C3, C3 to C5, J5 to J2, Q4 to Q1, R9 to R15, R10 to R16, R11 to R17, R19 to R18, R12 to R19, R13 to R20, R14 to R21, R15 to R22, R18 to R23, R31 to R24, SW41 to SW57, TP4 to TP2, TP2 to TP4, U4 to U3, U5 to U4

Commit message: remove global labels
Changed lines of the file:
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@@
 		)
 	)
-	(global_label "CHG"
+	(hierarchical_label "CHG"
 		(shape input)
 		(at 212.09 133.35 0)
@@
 			(justify left)
 		)
-		(property "Intersheetrefs" "${INTERSHEET_REFS}"
-			(at 218.9457 133.35 0)
-			(effects
-				(font
-					(size 1.27 1.27)
-				)
-				(justify left)
-				(hide yes)
-			)
-		)
 	)

Commit message: add bme280
Parts:
- TP4: footprint (none) -> TestPoint:TestPoint_Pad_D1.0mm
- renumbered R15 to R16, R16 to R17, R17 to R18, R18 to R19, R19 to R20, R20 to R21, R21 to R22, R22 to R23, R23 to R24, R24 to R25
