File: hardware/lcd.kicad_sch (KiCad schematic)
At the start: 7 parts, among them J3 Conn_01x40, Q3 AO3400A

Commit message: fix lcsc code for fpc (wrong but somewhat compatible footprint)
Parts:
- J3: LCSC C202114 -> C262674; LCSC_OLD (none) -> C202114
Changed lines of the file:
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@@
 			)
 		)
-		(property "LCSC" "C202114"
+		(property "LCSC_OLD" "C202114"
 			(at 138.43 86.36 0)
 			(effects
@@
 			(at 138.43 86.36 0)
 			(effects
+				(font
+					(size 1.27 1.27)
+				)
+				(hide yes)
+			)
+		)
+		(property "LCSC" "C262674"
+			(at 138.43 86.36 0)
+			(effects

Commit message: update lcsc codes to use (new?) basic components
Parts:
- R28, R29, R30: LCSC C116699 -> C21189
- R31: LCSC C105588 -> C22775
Changed lines of the file:
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@@
 			)
 		)
-		(property "LCSC" "C116699"
+		(property "LCSC" "C21189"
 			(at 83.82 175.26 0)
 			(effects
@@
 			)
 		)
-		(property "LCSC" "C116699"
+		(property "LCSC" "C21189"
 			(at 83.82 165.1 0)
 			(effects
@@
 			)
 		)
-		(property "LCSC" "C105588"
+		(property "LCSC" "C22775"
 			(at 46.99 107.95 0)
 			(effects
@@
 			)
 		)
-		(property "LCSC" "C116699"
+		(property "LCSC" "C21189"
 			(at 83.82 185.42 0)
 			(effects
